File: lofisampler.brd (EAGLE design)
At the start: 60 x 97.1 mm, 60 parts, among them IC1 ISD1820, IC2 78L05Z, IC3 LM358N

Commit message: Changed current limit resistors for the push buttons to 10k. Using 47k seems to deliver too small a current sometimes (some chips do not trigger on this).
Parts:
- R11, R7, R9: value 47k -> 10k
Changed lines of the file:
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@@
 <?xml version="1.0" encoding="utf-8"?>
 <!DOCTYPE eagle SYSTEM "eagle.dtd">
-<eagle version="8.5.1">
+<eagle version="9.0.1">
 <drawing>
 <settings>
-<setting alwaysvectorfont="no"/>
+<setting alwaysvectorfont="yes"/>
 <setting keepoldvectorfont="yes"/>
 <setting verticaltext="up"/>
@@
 <attribute name="VALUE" x="37.7952" y="17.7292" size="1.27" layer="27" ratio="10" rot="R90"/>
 </element>
-<element name="R11" library="rcl" library_urn="urn:adsk.eagle:library:334" package="0207/2V" package3d_urn="urn:adsk.eagle:package:23490/1" value="47k" x="46.99" y="33.02" smashed="yes">
+<element name="R11" library="rcl" library_urn="urn:adsk.eagle:library:334" package="0207/2V" package3d_urn="urn:adsk.eagle:package:23490/1" value="10k" x="46.99" y="33.02" smashed="yes">
 <attribute name="NAME" x="46.9392" y="34.036" size="1.27" layer="25" ratio="10"/>
 <attribute name="SPICEPREFIX" value="R" x="46.99" y="33.02" size="1.778" layer="27" display="off"/>
@@
 <attribute name="VALUE" x="49.8348" y="65.4558" size="1.27" layer="27" ratio="10" rot="R270"/>
 </element>
-<element name="R7" library="rcl" library_urn="urn:adsk.eagle:library:334" package="0207/2V" package3d_urn="urn:adsk.eagle:package:23490/1" value="47k" x="25.4" y="43.18" smashed="yes" rot="R180">
+<element name="R7" library="rcl" library_urn="urn:adsk.eagle:library:334" package="0207/2V" package3d_urn="urn:adsk.eagle:package:23490/1" value="10k" x="25.4" y="43.18" smashed="yes" rot="R180">
 <attribute name="NAME" x="24.8158" y="45.339" size="1.27" layer="25" ratio="10" rot="R180"/>
 <attribute name="SPICEPREFIX" value="R" x="25.4" y="43.18" size="1.778" layer="27" rot="R180" display="off"/>
@@
 <attribute name="VALUE" x="16.4592" y="20.6248" size="1.27" layer="27" ratio="10"/>
 </element>
-<element name="R9" library="rcl" library_urn="urn:adsk.eagle:library:334" package="0207/2V" package3d_urn="urn:adsk.eagle:package:23490/1" value="47k" x="33.02" y="31.115" smashed="yes">
+<element name="R9" library="rcl" library_urn="urn:adsk.eagle:library:334" package="0207/2V" package3d_urn="urn:adsk.eagle:package:23490/1" value="10k" x="33.02" y="31.115" smashed="yes">
 <attribute name="NAME" x="32.9692" y="32.131" size="1.27" layer="25" ratio="10"/>
 <attribute name="SPICEPREFIX" value="R" x="33.02" y="31.115" size="1.778" layer="27" display="off"/>

Commit message: latest updates
Parts:
- moved R21 7.85 mm to (47.0, 36.8)
- moved R15 7.41 mm to (12.7, 73.7), turned to 0 degrees
- moved R5 5.12 mm to (35.6, 64.8), turned to 180 degrees
- moved C3 4.26 mm to (50.8, 62.9)
- moved R24 3.59 mm to (35.6, 69.8), turned to 0 degrees
- moved R16 2.84 mm to (12.7, 68.6), turned to 180 degrees
- moved R20 1.90 mm to (47.0, 39.4), turned to 180 degrees
- moved R18 1.80 mm to (12.7, 71.1), turned to 180 degrees
- moved C2 1.80 mm to (38.1, 60.3), turned to 270 degrees
- moved R6 1.80 mm to (50.8, 66.7), turned to 0 degrees
- moved R23 1.80 mm to (35.6, 67.3)
- moved R25 1.80 mm to (35.6, 72.4)
- moved R11 1.27 mm to (47.0, 34.3)
- moved D4 0.64 mm to (35.6, 9.53)
- moved R19 0.63 mm to (47.0, 41.9)
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Routing:
- net N$20: track 17.4 -> 8.69 mm
- net N$22: track 33.2 -> 25.6 mm
- net N$33: track 14.8 -> 7.62 mm
- net N$16: track 73.1 -> 67.3 mm
- net N$12: track 13.0 -> 7.40 mm
- net N$32: track 26.8 -> 21.8 mm
- net N$15: track 46.2 -> 50.8 mm
- net N$14: track 3.18 -> 7.51 mm
- net N$10: track 8.06 -> 12.1 mm
- net N$31: track 80.6 -> 76.5 mm
- net PLAY_L: track 35.3 -> 39.0 mm
- net N$25: track 13.5 -> 9.94 mm
- net N$8: track 6.28 -> 3.37 mm
- net N$17: track 10.2 -> 13.0 mm
- net N$30: track 3.65 -> 4.92 mm
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Other:
- board text added: "ISD1820 sampler/filter/distortion"
- board text removed: "ISD1820 sampler/bitcrusher/filter"
